File: ui.kicad_sch (KiCad schematic)
At the start: 22 parts, among them Q2 BJT 2222A, SW1 Primary Button, SW3 Secondary Button, U9 X096-2864KSWPG01-H30

Commit message: Add test points to schematic.
Parts:
- added TP14: TP_CS, symbol Connector:TestPoint
- added TP16: TP_MOTOR, symbol Connector:TestPoint
Connections:
- net CS: now also TP14.1
- net VIB_MOTOR: now also TP16.1
Changed lines of the file:
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@@
+		)
+	)
+	(label "CS"
+		(at 227.33 149.86 270)
+		(effects
+			(font
+				(size 1.27 1.27)
+			)
+			(justify right bottom)
 		)
 	)
 	(label "DC"
 		(at 156.21 74.93 180)
+		(effects
+			(font
+				(size 1.27 1.27)
+			)
+			(justify right bottom)
+		)
+	)
+	(label "VIB_MOTOR"
+		(at 215.9 149.86 270)
 		(effects
 			(font
@@
 	)
 	(symbol
+		(lib_id "Connector:TestPoint")
+		(at 227.33 149.86 0)
+		(unit 1)
+		(body_style 1)
+		(exclude_from_sim no)
+		(in_bom yes)
+		(on_board yes)
+		(in_pos_files yes)
+		(dnp no)
+		(property "Reference" "TP14"
+			(at 224.536 141.478 0)
+			(show_name no)
+			(do_not_autoplace no)
+			(effects
+				(font
+					(size 1.27 1.27)
+				)
+				(justify left)
+			)
+		)
+		(property "Value" "TP_CS"
+			(at 224.536 144.018 0)
+			(show_name no)
+			(do_not_autoplace no)
+			(effects
+				(font
+					(size 1.27 1.27)
+				)
+				(justify left)
+			)
+		)
+		(property "Footprint" ""
+			(at 232.41 149.86 0)
+			(hide yes)
+			(show_name no)
+			(do_not_autoplace no)
+			(effects
+				(font
+					(size 1.27 1.27)
+				)
+			)
+		)
+		(property "Datasheet" ""
+			(at 232.41 149.86 0)
+			(hide yes)
+			(show_name no)
+			(do_not_autoplace no)
+			(effects
+				(font
+					(size 1.27 1.27)
+				)
+			)
+		)
+		(property "Description" "test point"
+			(at 227.33 149.86 0)
+			(hide yes)
+			(show_name no)
+			(do_not_autoplace no)
+			(effects
+				(font
+					(size 1.27 1.27)
+				)
+			)
+		)
+		(pin "1"
+		)
+		(instances
+			(project "pdn-kit-hardware"
+				(path "/7ba8b3ae-d553-4981-99e4-6a44bc3bbf14/9dfd9d22-8a53-42e3-bd85-2d3ea20f3dc4"
+					(reference "TP14")
+					(unit 1)
+				)
+			)
+		)
+	)
+	(symbol
 		(lib_id "global:X096-2864KSWPG01-H30")
 		(at 196.85 76.2 0)
@@
 					(unit 1)
 				)
+			)
+		)
+	)
+	(symbol
+		(lib_id "Connector:TestPoint")
+		(at 215.9 149.86 0)
+		(unit 1)
+		(body_style 1)
+		(exclude_from_sim no)
+		(in_bom yes)
+		(on_board yes)
+		(in_pos_files yes)
+		(dnp no)
+		(property "Reference" "TP16"
+			(at 212.598 140.97 0)
+			(show_name no)
+			(do_not_autoplace no)
+			(effects
+				(font
+					(size 1.27 1.27)
+				)
+				(justify left)
+			)
+		)
+		(property "Value" "TP_MOTOR"
+			(at 212.598 143.51 0)
+			(show_name no)
+			(do_not_autoplace no)
+			(effects
+				(font
+					(size 1.27 1.27)
+				)
+				(justify left)
+			)
+		)
+		(property "Footprint" ""
+			(at 220.98 149.86 0)
+			(hide yes)
+			(show_name no)
+			(do_not_autoplace no)
+			(effects
+				(font
+					(size 1.27 1.27)
+				)
+			)
+		)
+		(property "Datasheet" ""
+			(at 220.98 149.86 0)
+			(hide yes)
+			(show_name no)
+			(do_not_autoplace no)
+			(effects
+				(font
+					(size 1.27 1.27)
+				)
+			)
+		)
+		(property "Description" "test point"
+			(at 215.9 149.86 0)
+			(hide yes)
+			(show_name no)
+			(do_not_autoplace no)
+			(effects
+				(font
+					(size 1.27 1.27)
+				)
+			)
+		)
+		(pin "1"
+		)
+		(instances
+			(project "pdn-kit-hardware"
+				(path "/7ba8b3ae-d553-4981-99e4-6a44bc3bbf14/9dfd9d22-8a53-42e3-bd85-2d3ea20f3dc4"
+					(reference "TP16")
+					(unit 1)
+				)

Commit message: Add extracted data sheets to project.
Parts:
- C1P1, C2P2: value 1uF -> 1 uF
- C_Motor1, C_VCC1, C_VDD1: value 100nF -> 100 nF
- C_VCC2, C_VDD2: value 4.7uF -> 4.7 uF
Changed lines of the file:
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@@
 			)
 		)
-		(property "Value" "100nF"
+		(property "Value" "100 nF"
 			(at 54.61 41.275 0)
 			(show_name no)
@@
 			)
 		)
-		(property "Value" "4.7uF"
+		(property "Value" "4.7 uF"
 			(at 118.364 113.03 0)
 			(show_name no)
@@
 			)
 		)
-		(property "Value" "1uF"
+		(property "Value" "1 uF"
 			(at 173.99 36.83 90)
 			(show_name no)
@@
 			)
 		)
-		(property "Value" "100nF"
+		(property "Value" "100 nF"
 			(at 139.7 113.0299 0)
 			(show_name no)
@@
 			)
 		)
-		(property "Value" "1uF"
+		(property "Value" "1 uF"
 			(at 166.37 41.91 90)
 			(show_name no)
@@
 			)
 		)
-		(property "Value" "100nF"
+		(property "Value" "100 nF"
 			(at 139.7 64.7699 0)
 			(show_name no)
@@
 			)
 		)
-		(property "Value" "4.7uF"
+		(property "Value" "4.7 uF"
 			(at 118.872 64.77 0)
 			(show_name no)

Commit message: Fix LED's -> anode wired to VCC, not GND.
Changed lines of the file:
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@@
 		(property "Value" "GND"
 			(at 156.21 119.38 0)
+			(hide yes)
 			(show_name no)
 			(do_not_autoplace no)
@@
 		(property "Value" "GND"
 			(at 147.32 57.15 0)
+			(hide yes)
 			(show_name no)
 			(do_not_autoplace no)
@@
 		(property "Value" "GND"
 			(at 41.91 58.42 0)
+			(hide yes)
 			(show_name no)
 			(do_not_autoplace no)
@@
 		(property "Value" "GND"
 			(at 133.35 72.39 0)
+			(hide yes)
 			(show_name no)
 			(do_not_autoplace no)
@@
 		(property "Value" "GND"
 			(at 38.1 86.36 0)
+			(hide yes)
 			(show_name no)
 			(do_not_autoplace no)
@@
 		(property "Value" "GND"
 			(at 80.01 86.36 0)
+			(hide yes)
 			(show_name no)
 			(do_not_autoplace no)
@@
 		(property "Value" "GND"
 			(at 184.15 57.1499 90)
+			(hide yes)
 			(show_name no)
 			(do_not_autoplace no)
@@
 		(property "Value" "GND"
 			(at 133.35 120.65 0)
+			(hide yes)
 			(show_name no)
 			(do_not_autoplace no)
@@
 		(property "Value" "GND"
 			(at 184.15 39.3699 90)
-			(show_name no)
-			(do_not_autoplace no)
+			(hide yes)
+			(show_name no)
+			(do_not_autoplace no)
